Commit message: feat(urdf update)

File: urdf/linear_actuator.xacro (robot description, xacro)
@@ -18,5 +18,5 @@
         <parent link="${name}_holder"/>
         <child link="${name}_up_tensor"/>
-        <origin xyz="0 0 -0.013" rpy="0 0 0" />
+        <origin xyz="0 0 -0.0175" rpy="0 0 0" /> <!-- half universal join = 13 mm, nut = 4 mm, whasher = 0.5 mm -->
     </joint>
     <link name="${name}_down_tensor"/>
@@ -24,5 +24,5 @@
         <parent link="${name}_base"/>
         <child link="${name}_down_tensor"/>
-        <origin xyz="0 0 0.013" rpy="0 0 0" />
+        <origin xyz="0 0 0.0175" rpy="0 0 0" /> <!-- half universal join = 13 mm, nut = 4 mm, whasher = 0.5 mm -->
     </joint>
     <xacro:include filename="$(find robotic_neck_viz)/urdf/cross_piece.xacro"/>
@@ -51,5 +51,5 @@
         <parent link="${name}_linear_actuator_axis"/>
         <child link="${name}_linear_actuator_tube"/>
-        <origin xyz="0 0 0.149" rpy="0 0 0"/>
+        <origin xyz="0 0 0.1645" rpy="0 0 0"/> <!-- origin tensor len = (pilar_len(172) + UJ_p(23) + nut(4) + whasher(5)))-(universal join(26) + 2*(nut(4) + whasher(5)))-= 172 - 3 - 4.5- = 164,5 mm -->
         <axis xyz="0 0 1"/>
         <limit lower="-0.017" upper="0.063" effort="100" velocity="0.01"/>

File: urdf/robotic_neck.urdf.xacro (robot description, xacro)
@@ -5,5 +5,5 @@
     <link name="base_link">
       <visual>
-          <origin xyz="-0.015 0 -0.173" rpy="0 0 ${pi}"/>
+          <origin xyz="-0.015 0 -0.193" rpy="0 0 ${pi}"/>
           <geometry>
               <mesh filename="package://robotic_neck_viz/urdf/models/base/mesh/base.dae" />
@@ -14,5 +14,5 @@
         <parent link="world"/>
         <child link="base_link"/>
-        <origin xyz="0 0 0.1635" rpy="0 0 0" />
+        <origin xyz="0 0 0.1835" rpy="0 0 0" />
     </joint>
     <xacro:include filename="$(find robotic_neck_viz)/urdf/cross_piece.xacro"/>
@@ -29,5 +29,5 @@
       <parent link="main_cross_piece_roll"/>
       <child link="platform"/>
-      <origin xyz="0 0 0.0115"/>
+      <origin xyz="0 0 0.016"/> <!-- half universal join = 11,5 mm, nut = 4 mm, whasher = 0.5 mm -->
     </joint>
     <xacro:include filename="$(find robotic_neck_viz)/urdf/linear_actuator.xacro"/>

Commit message: update

File: urdf/linear_actuator.xacro (robot description, xacro)
@@ -4,7 +4,7 @@
     <link name="${namespace}/${name}_base"/>
     <joint name="${namespace}/${name}_base_joint" type="fixed">
-        <parent link="world"/>
+        <parent link="${namespace}/base_link"/>
         <child link="${namespace}/${name}_base"/>
-        <origin xyz="-0.075 ${side*0.05} 0" rpy="0 0 0" />
+        <origin xyz="-0.075 ${side*0.05} -0.1835" rpy="0 0 0" />
     </joint>
     <link name="${namespace}/${name}_holder"/>

File: urdf/robotic_neck.xacro (robot description, xacro)
@@ -2,7 +2,6 @@
 <!-- Basic WAM-V with gazebo plugins for dynamics -->
 <robot xmlns:xacro="http://ros.org/wiki/xacro">
-    <xacro:macro name="robotic_neck" params="namespace color">
-      <link name="world"/>
-      <link name="base_link">
+    <xacro:macro name="robotic_neck" params="namespace color parent_frame">
+      <link name="${namespace}/base_link">
         <visual>
             <origin xyz="-0.015 0 -0.193" rpy="0 0 ${pi}"/>
@@ -12,11 +11,11 @@
         </visual>
       </link>
-      <joint name="base_link_joint" type="fixed">
-          <parent link="world"/>
-          <child link="base_link"/>
+      <joint name="${namespace}/base_link_joint" type="fixed">
+          <parent link="${parent_frame}"/>
+          <child link="${namespace}/base_link"/>
           <origin xyz="0 0 0.1835" rpy="0 0 0" />
       </joint>
       <xacro:include filename="$(find robotic_neck_viz)/urdf/cross_piece.xacro"/>
-      <xacro:cross_piece name="main" namespace="${namespace}" parent="base_link" rot1="pitch" rot2="roll" pitch2roll="1"/>
+      <xacro:cross_piece name="main" namespace="${namespace}" parent="${namespace}/base_link" rot1="pitch" rot2="roll" pitch2roll="1"/>
       <link name="${namespace}/platform">
       <visual>

File: urdf/robotic_neck_cam.xacro (robot description, xacro)
@@ -2,8 +2,9 @@
 <!-- Basic WAM-V with gazebo plugins for dynamics -->
 <robot xmlns:xacro="http://ros.org/wiki/xacro">
-    <xacro:macro name="robotic_neck" params="namespace color">
+    <xacro:macro name="robotic_neck" params="namespace color parent_frame
+                                             x=0.0 y=0.0 z=0.1835
+                                             R=0.0 P=0.0 Y=0.0">
       <!-- ADD BASE LINK-->
-      <link name="world"/>
-      <link name="base_link">
+      <link name="${namespace}/base_link">
         <visual>
             <origin xyz="-0.015 0 -0.193" rpy="0 0 ${pi}"/>
@@ -13,11 +14,11 @@
         </visual>
       </link>
-      <joint name="base_link_joint" type="fixed">
-          <parent link="world"/>
-          <child link="base_link"/>
-          <origin xyz="0 0 0.1835" rpy="0 0 0" />
+      <joint name="${namespace}/base_link_joint" type="fixed">
+          <parent link="${parent_frame}"/>
+          <child link="${namespace}/base_link"/>
+          <origin xyz="${x} ${y} ${z}" rpy="${R} ${P} ${Y}" />
       </joint>
       <xacro:include filename="$(find robotic_neck_viz)/urdf/cross_piece.xacro"/>
-      <xacro:cross_piece name="main" namespace="${namespace}" parent="base_link" rot1="pitch" rot2="roll" pitch2roll="1"/>
+      <xacro:cross_piece name="main" namespace="${namespace}" parent="${namespace}/base_link" rot1="pitch" rot2="roll" pitch2roll="1"/>
       <!-- ADD PLATFORM-->
       <link name="${namespace}/platform">

File: urdf/robotic_neck_state.urdf.xacro (robot description, xacro)
@@ -2,5 +2,5 @@
 <!-- Basic WAM-V with gazebo plugins for dynamics -->
 <robot xmlns:xacro="http://ros.org/wiki/xacro" name="robotic_neck">
-    <xacro:arg name="camera_enabled" default="false"/>
+    <xacro:arg name="camera_enabled" default="true"/>
     <xacro:if value="$(arg camera_enabled)">
         <xacro:include filename="$(find robotic_neck_viz)/urdf/robotic_neck_cam.xacro"/>
@@ -9,4 +9,5 @@
         <xacro:include filename="$(find robotic_neck_viz)/urdf/robotic_neck.xacro"/>
     </xacro:unless>
-    <xacro:robotic_neck namespace="state" color="_white"/>
+    <link name="world"/>
+    <xacro:robotic_neck namespace="state" color="_white" parent_frame="world"/>
 </robot>

File: urdf/robotic_neck_target.urdf.xacro (robot description, xacro)
@@ -3,4 +3,5 @@
 <robot xmlns:xacro="http://ros.org/wiki/xacro" name="robotic_neck">
     <xacro:include filename="$(find robotic_neck_viz)/urdf/robotic_neck.xacro"/>
-    <xacro:robotic_neck namespace="target" color=""/>
+    <link name="world"/>
+    <xacro:robotic_neck namespace="target" color="" parent_frame="world"/>
 </robot>

File: urdf/wamv_robotic_neck.urdf.xacro (robot description, xacro)
@@ -4,14 +4,10 @@
   <xacro:property name="cfg_file" value="$(find robotic_neck_viz)/config/robot_urdf.yaml" />
   <xacro:property name="cfg" value="${xacro.load_yaml(cfg_file)}"/>
-  <xacro:arg name="lidar_enabled" default="${cfg['lidar_enabled']}" />
-  <xacro:arg name="lidar_namespace" default="${cfg['lidar_namespace']}"/>
   <xacro:arg name="namespace" default="${cfg['namespace']}"/>
-  <xacro:property name="lidar_namespace" value="$(arg lidar_namespace)" scope="global" />
   <xacro:property name="namespace" value="$(arg namespace)" scope="global" />
   <!-- === The WAM-V platform === -->
   <xacro:include filename="$(find caleuche_viz)/urdf/components/wamv/wamv.urdf.xacro"/>
-  <!-- Add 3D LIDAR -->
-  <xacro:if value="$(arg lidar_enabled)">
-    <xacro:include filename="$(find robotic_neck_viz)/urdf/lidar/ouster_lidar.xacro"/>
-  </xacro:if>
+  <!-- === ADD Robotic Neck === -->
+  <xacro:include filename="$(find robotic_neck_viz)/urdf/robotic_neck_cam.xacro"/>
+  <xacro:robotic_neck namespace="state" color="_white" parent_frame="wamv/base_link" x="0.55" z="1.5"/>
 </robot>
